Commit message: parallel hill climber with specified number of generations

File: body.urdf (robot description, URDF)
Before this commit: robot robot, 3 links, 2 joints
Links:
- removed link Back_Leg
- removed link Front_Leg
- added link BackLeg, mass 1; collision box size=1 1 1; visual box size=1 1 1
- added link FrontLeg, mass 1; collision box size=1 1 1; visual box size=1 1 1
Joints:
- joint Torso_BackLeg: child Back_Leg -> BackLeg; origin xyz=-0.5 0 1 rpy=0 0 0 -> xyz=0.5 0 1 rpy=0 0 0
- joint Torso_FrontLeg: child Front_Leg -> FrontLeg; origin xyz=0.5 0 1 rpy=0 0 0 -> xyz=1.5 0 1 rpy=0 0 0
